File: Circuit/V1/Water Board.kicad_pcb (KiCad board)
At the start: 2 copper layers, 76.2 x 48.3 mm, 30 parts, among them J1 Pump Header, J2 Tank 1 Header, J3 Tank 2 Header, J4 Water Temp Header, J5 Water Level Header, J6 Water Level V Seletor Header, J7 Barrel_Jack, M1 MountingHole_2.2mm_M2_DIN965_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, M2 MountingHole_2.2mm_M2_DIN965_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, M3 MountingHole_2.2mm_M2_DIN965_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

Commit message: Added pull down resistors to mosfets
Parts:
- added R10: 10K, Resistor_SMD:R_0805_2012Metric_Pad1.20x1.40mm_HandSolder, F.Cu at (61.0, 66.0)
- added R8: 10k, Resistor_SMD:R_0805_2012Metric_Pad1.20x1.40mm_HandSolder, F.Cu at (96.2, 66.0)
- added R9: 10k, Resistor_SMD:R_0805_2012Metric_Pad1.20x1.40mm_HandSolder, F.Cu at (91.8, 69.8)
- D7: footprint PCM_Diode_SMD_AKL:D_SMA -> PCM_Diode_SMD_Handsoldering_AKL:D_SMA_BigPads
- J6: value Water Level V Seletor Header -> Water Level Voltage Selector
- Q1, Q2, Q3: footprint PCM_Package_TO_SOT_SMD_AKL:SOT-23 -> PCM_Package_TO_SOT_SMD_AKL:SOT-23_BigPads
- R7: value 10K -> 10k
- moved R7 26.1 mm to (85.7, 74.3)
- moved R2 3.78 mm to (96.2, 64.1), turned to 180 degrees
- moved R3 3.55 mm to (91.8, 67.9), turned to 0 degrees
- moved Q1 1.31 mm to (91.4, 74.5)
- moved Q3 0.63 mm to (97.8, 71.4)
- moved Q2 0.63 mm to (96.9, 59.8)
- moved D5 0.56 mm to (100.3, 64.1)
- moved R5 0.56 mm to (100.3, 66.0)
- moved D6 0.27 mm to (100.1, 80.0)
- moved R6 0.27 mm to (100.1, 81.9)
Connections:
- R7 pad 1: /dallas -> GND
- R7 pad 2: +3V3 -> /pump_enable
Routing:
- net GND: track 4.56 -> 10.6 mm, vias 18 -> 15
- net /tank_2_enable: track 47.1 -> 51.7 mm
- net Net-(Q2-G): track 5.67 -> 9.22 mm
- net /pump_enable: track 31.8 -> 34.5 mm
- net /tank_1_enable: track 46.5 -> 44.6 mm
- net Net-(Q3-G): track 8.72 -> 7.32 mm
- net Net-(D1-A): track 8.64 -> 9.45 mm
- net Net-(Q1-G): track 6.75 -> 7.54 mm

Commit message: Revise resistor and LED layout, Added preview images
Parts:
- moved R6 12.1 mm to (100.1, 69.8)
- moved D6 8.26 mm to (100.1, 71.8)
- moved R3 5.78 mm to (96.2, 71.8), turned to 180 degrees
- moved Q3 5.25 mm to (97.2, 76.6)
- moved R9 4.35 mm to (96.2, 69.8), turned to 180 degrees
- moved D5 0.25 mm to (100.1, 64.1)
- moved R5 0.25 mm to (100.1, 66.0)
- moved Q2 0.17 mm to (96.8, 59.8)
Routing:
- net /tank_2_enable: track 51.7 -> 44.0 mm
- net +24V: track 115.4 -> 117.4 mm
- net Net-(D3-A): track 12.2 -> 10.2 mm
- net Net-(Q3-G): track 7.32 -> 5.37 mm
- net GND: track 10.6 -> 9.96 mm
